File: hw/pcb/logger.kicad_pcb (KiCad board)
At the start: 2 copper layers, 42 x 46.6 mm, 70 parts, among them J1 BAT+, J2 SWO, J3 DEBUG, J4 USB_B_Micro, J5 ANT1575-2006B, J6 OLED-128O064D, J7 BAT-, Q1 DMG1012UW, Q2 DMG2307L, SW1 Next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

Commit message: Added value to crystal caps
Parts:
- C2, C3: value C -> 6p8
Connections:
- J2 pad 6: (no net) -> Net-(J2-Pad6)
- J6 pad 16: (no net) -> Net-(J6-Pad16)
- J6 pad 17: (no net) -> Net-(J6-Pad17)
- J6 pad 21: (no net) -> Net-(J6-Pad21)
- J6 pad 22: (no net) -> Net-(J6-Pad22)
- J6 pad 23: (no net) -> Net-(J6-Pad23)
- J6 pad 24: (no net) -> Net-(J6-Pad24)
- J6 pad 25: (no net) -> Net-(J6-Pad25)
- J6 pad 7: (no net) -> Net-(J6-Pad7)
- U1 pad 11: (no net) -> Net-(U1-Pad11)
- U1 pad 18: (no net) -> Net-(U1-Pad18)
- U1 pad 19: (no net) -> Net-(U1-Pad19)
- U1 pad 2: (no net) -> Net-(U1-Pad2)
- U1 pad 20: (no net) -> Net-(U1-Pad20)
- U1 pad 21: (no net) -> Net-(U1-Pad21)
- U1 pad 22: (no net) -> Net-(U1-Pad22)
- U1 pad 27: (no net) -> Net-(U1-Pad27)
- U1 pad 28: (no net) -> Net-(U1-Pad28)
- U1 pad 29: (no net) -> Net-(U1-Pad29)
- U1 pad 3: (no net) -> Net-(U1-Pad3)
- U1 pad 40: (no net) -> Net-(U1-Pad40)
- U2 pad 11: (no net) -> Net-(U2-Pad11)
- U2 pad 12: (no net) -> Net-(U2-Pad12)
- U5 pad 13: (no net) -> Net-(U5-Pad13)
- U5 pad 14: (no net) -> Net-(U5-Pad14)
- U5 pad 15: (no net) -> Net-(U5-Pad15)
- U5 pad 16: (no net) -> Net-(U5-Pad16)
- U5 pad 17: (no net) -> Net-(U5-Pad17)
- U5 pad 18: (no net) -> Net-(U5-Pad18)
- U5 pad 4: (no net) -> Net-(U5-Pad4)
- U5 pad 5: (no net) -> Net-(U5-Pad5)
